Commit message: upload robot with sensors integrated

File: src/my_robot/urdf/my_robot.xacro (robot description, xacro)
@@ -2,4 +2,5 @@
 <robot name="my_robot" xmlns:xacro="http://www.ros.org/wiki/xacro">
   <link name="robot_footprint"></link>
+  <xacro:include filename="$(find my_robot)/urdf/my_robot.gazebo" />
   <joint name="robot_footprint_joint" type="fixed">
     <origin xyz="0 0 0" rpy="0 0 0" />
@@ -78,4 +79,12 @@
     </visual>
   </link>
+  <joint type="continuous" name="right_wheel_hinge">
+    <origin xyz="0 -0.15 0" rpy="0 0 0"/>
+    <child link="right_wheel"/>
+    <parent link="chassis"/>
+    <axis xyz="0 1 0" rpy="0 0 0"/>
+    <limit effort="10000" velocity="1000"/>
+    <dynamics damping="1.0" friction="1.0"/>
+  </joint>
   <link name='left_wheel'>
     <inertial>
@@ -109,13 +118,4 @@
     <dynamics damping="1.0" friction="1.0"/>
   </joint>
-  <joint type="continuous" name="right_wheel_hinge">
-    <origin xyz="0 -0.15 0" rpy="0 0 0"/>
-    <child link="right_wheel"/>
-    <parent link="chassis"/>
-    <axis xyz="0 1 0" rpy="0 0 0"/>
-    <limit effort="10000" velocity="1000"/>
-    <dynamics damping="1.0" friction="1.0"/>
-  </joint>
-  <!-- Sensors -->
   <link name='camera'>
     <inertial>
@@ -166,6 +166,5 @@
       <origin xyz="0 0 0" rpy=" 0 0 0"/>
       <geometry>
-        <box size="0.1 0.1 0.1"/>
-        <!-- <mesh filename=“package://my_robot/meshes/hokuyo.dae”/> -->
+        <mesh filename="package://my_robot/meshes/hokuyo.dae"/>
       </geometry>
     </visual>
@@ -178,4 +177,7 @@
   </joint>
   <!-- Material Descriptions -->
+  <gazebo reference="chassis">
+      <material>Gazebo/Blue</material>
+  </gazebo>
   <gazebo reference="left_wheel">
     <material>Gazebo/Green</material>
@@ -184,9 +186,6 @@
       <material>Gazebo/Green</material>
   </gazebo>
-  <gazebo reference="chassis">
+  <gazebo reference="camera">
       <material>Gazebo/Red</material>
   </gazebo>
-  <gazebo reference="camera">
-      <material>Gazebo/Blue</material>
-  </gazebo>
 </robot>

Commit message: solve project 2

File: src/my_robot/urdf/my_robot.xacro (robot description, xacro)
@@ -22,5 +22,5 @@
       <origin xyz="0 0 0" rpy=" 0 0 0"/>
       <geometry>
-        <box size=".4 .2 .1"/>
+        <box size=".2 .2 .1"/>
       </geometry>
     </collision>
@@ -28,21 +28,9 @@
       <origin xyz="0 0 0" rpy=" 0 0 0"/>
       <geometry>
-        <box size=".4 .2 .1"/>
-      </geometry>
-    </visual>
-    <collision name='back_caster_collision'>
-      <origin xyz="-0.15 0 -0.05" rpy=" 0 0 0"/>
-      <geometry>
-        <sphere radius="0.0499"/>
-      </geometry>
-    </collision>
-    <visual name='back_caster_visual'>
-      <origin xyz="-0.15 0 -0.05" rpy=" 0 0 0"/>
-      <geometry>
-        <sphere radius="0.05"/>
+        <box size=".2 .2 .1"/>
       </geometry>
     </visual>
     <collision name='front_caster_collision'>
-      <origin xyz="0.15 0 -0.05" rpy=" 0 0 0"/>
+      <origin xyz="0.1 0 -0.05" rpy=" 0 0 0"/>
       <geometry>
         <sphere radius="0.0499"/>
@@ -50,5 +38,5 @@
     </collision>
     <visual name='front_caster_visual'>
-      <origin xyz="0.15 0 -0.05" rpy=" 0 0 0"/>
+      <origin xyz="0.1 0 -0.05" rpy=" 0 0 0"/>
       <geometry>
         <sphere radius="0.05"/>
@@ -59,5 +47,5 @@
     <inertial>
         <mass value="5.0"/>
-        <origin xyz="0.0 0 0" rpy=" 0 0 0"/>
+        <origin xyz="0 0 0" rpy=" 0 0 0"/>
         <inertia
             ixx="0.1" ixy="0" ixz="0"
@@ -80,5 +68,5 @@
   </link>
   <joint type="continuous" name="right_wheel_hinge">
-    <origin xyz="0 -0.15 0" rpy="0 0 0"/>
+    <origin xyz="-0.05 -0.1 0" rpy="0 0 0"/>
     <child link="right_wheel"/>
     <parent link="chassis"/>
@@ -111,5 +99,5 @@
   </link>
   <joint type="continuous" name="left_wheel_hinge">
-    <origin xyz="0 0.15 0" rpy="0 0 0"/>
+    <origin xyz="-0.05 0.1 0" rpy="0 0 0"/>
     <child link="left_wheel"/>
     <parent link="chassis"/>
@@ -142,5 +130,5 @@
   </link>
   <joint type="fixed" name="camera_joint">
-    <origin xyz="0.2 0 0" rpy="0 0 0"/>
+    <origin xyz="0.1 0 0.05" rpy="0 0 0"/>
     <child link="camera"/>
     <parent link="chassis"/>
@@ -171,5 +159,5 @@
   </link>
   <joint type="fixed" name="hokuyo_joint">
-    <origin xyz="0.15 0 0.1" rpy="0 0 0"/>
+    <origin xyz="0.0 0 0.1" rpy="0 0 0"/>
     <child link="hokuyo"/>
     <parent link="chassis"/>

Commit message: setup project 4

File: src/my_robot/urdf/my_robot.xacro (robot description, xacro)
@@ -164,4 +164,11 @@
     <axis xyz="0 1 0" rpy="0 0 0"/>
   </joint>
+  <!-- <joint name="camera_optical_joint" type="fixed">
+    <origin xyz="0.1 0 0.1" rpy="-1.5707 0 -1.5707"/>
+    <parent link="chassis"/>
+    <child link="camera_link_optical"/>
+  </joint>
+  <link name="camera_link_optical">
+  </link> -->
   <!-- Material Descriptions -->
   <gazebo reference="chassis">

Commit message: upload the last changes

File: src/my_robot/urdf/my_robot.xacro (robot description, xacro)
@@ -164,11 +164,11 @@
     <axis xyz="0 1 0" rpy="0 0 0"/>
   </joint>
-  <!-- <joint name="camera_optical_joint" type="fixed">
+  <joint name="camera_optical_joint" type="fixed">
     <origin xyz="0.1 0 0.1" rpy="-1.5707 0 -1.5707"/>
-    <parent link="chassis"/>
+    <parent link="camera"/>
     <child link="camera_link_optical"/>
   </joint>
   <link name="camera_link_optical">
-  </link> -->
+  </link>
   <!-- Material Descriptions -->
   <gazebo reference="chassis">
